Commit message: Add changes flow with updated poses

File: yumi_description/urdf/Grippers/yumi_servo_gripper.xacro (robot description, xacro)
@@ -57,5 +57,5 @@
         <origin xyz="0 0 0" rpy="0 0 0"/>
         <geometry>
-          <mesh filename="package://yumi_description/meshes/gripper/finger.stl"/>
+          <mesh filename="package://yumi_description/meshes/gripper/SPL_Yumi_Right_Finger.stl"/>
         </geometry>
         <material name="Blue"/>
@@ -64,5 +64,5 @@
         <origin xyz="0 0 0" rpy="0 0 0"/>
         <geometry>
-          <mesh filename="package://yumi_description/meshes/gripper/coarse/finger.stl"/>
+          <mesh filename="package://yumi_description/meshes/gripper/SPL_Yumi_Right_Finger.stl"/>
         </geometry>
         <material name="Blue"/>
@@ -89,5 +89,5 @@
         <origin xyz="0 0 0" rpy="0 0 0"/>
         <geometry>
-          <mesh filename="package://yumi_description/meshes/gripper/finger.stl"/>
+          <mesh filename="package://yumi_description/meshes/gripper/SPL_Yumi_Left_Finger.stl"/>
         </geometry>
         <material name="Blue"/>
@@ -96,5 +96,5 @@
         <origin xyz="0 0 0" rpy="0 0 0"/>
         <geometry>
-          <mesh filename="package://yumi_description/meshes/gripper/coarse/finger.stl"/>
+          <mesh filename="package://yumi_description/meshes/gripper/SPL_Yumi_Left_Finger.stl"/>
         </geometry>
         <material name="Blue"/>

File: yumi_description/urdf/yumi_custom.urdf (robot description, URDF)
Before this commit: robot yumi, 23 links, 22 joints
Links:
- link gripper_l_finger_l: geometry collision mesh filename=package://yumi_description/meshes/gripper/coarse/finger.stl; visual mesh filename=package://yumi_description/meshes/gripper/SPL_Yumi_Left_Fin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
- link gripper_l_finger_r: geometry collision mesh filename=package://yumi_description/meshes/gripper/coarse/finger.stl; visual mesh filename=package://yumi_description/meshes/gripper/SPL_Yumi_Left_Fin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

Commit message: Fixed last commit, removing catkin_ws, with changes to the Yumi Gripper (custom for SPL). Fixed Dockerfile workspace set up (rep clones)

File: yumi_description/urdf/Grippers/yumi_servo_gripper.xacro (robot description, xacro)
@@ -57,5 +57,5 @@
         <origin xyz="0 0 0" rpy="0 0 0"/>
         <geometry>
-          <mesh filename="package://yumi_description/meshes/gripper/SPL_Yumi_Right_Finger.stl"/>
+          <mesh filename="package://yumi_description/meshes/gripper/finger.stl"/>
         </geometry>
         <material name="Blue"/>
@@ -64,5 +64,5 @@
         <origin xyz="0 0 0" rpy="0 0 0"/>
         <geometry>
-          <mesh filename="package://yumi_description/meshes/gripper/SPL_Yumi_Right_Finger.stl"/>
+          <mesh filename="package://yumi_description/meshes/gripper/coarse/finger.stl"/>
         </geometry>
         <material name="Blue"/>
@@ -89,5 +89,5 @@
         <origin xyz="0 0 0" rpy="0 0 0"/>
         <geometry>
-          <mesh filename="package://yumi_description/meshes/gripper/SPL_Yumi_Left_Finger.stl"/>
+          <mesh filename="package://yumi_description/meshes/gripper/finger.stl"/>
         </geometry>
         <material name="Blue"/>
@@ -96,5 +96,5 @@
         <origin xyz="0 0 0" rpy="0 0 0"/>
         <geometry>
-          <mesh filename="package://yumi_description/meshes/gripper/SPL_Yumi_Left_Finger.stl"/>
+          <mesh filename="package://yumi_description/meshes/gripper/coarse/finger.stl"/>
         </geometry>
         <material name="Blue"/>

File: yumi_description/urdf/yumi.urdf (robot description, URDF)
Before this commit: robot yumi, 23 links, 22 joints
Links:
- link gripper_r_finger_l: geometry collision mesh filename=package://yumi_description/meshes/gripper/SPL_Yumi_Left_Fin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; visual mesh filename=package://yumi_description/meshes/gripper/SPL_Yumi_Left_Fin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
- link gripper_r_finger_r: geometry collision mesh filename=package://yumi_description/meshes/gripper/SPL_Yumi_Right_Fi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; visual mesh filename=package://yumi_description/meshes/gripper/SPL_Yumi_Right_Fi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

Commit message: Added TCP for both grippers both in generated urdf and gripper xacros. Changed SRDF for these new TCP links, added links to arm groups for ease of association. Added Group ROSAPI and parsing functions, with a group change (call moveit_commander's switch). TODO: adjust offsets for new TCPs (probably the math)

File: yumi_description/urdf/Grippers/yumi_servo_gripper.xacro (robot description, xacro)
@@ -101,4 +101,23 @@
       </collision>
     </link>
+    <link name="${name}_tcp">
+    <!-- NO visual, NO collision, NO inertial - it's purely virtual! -->
+    <!-- Or optionally add a tiny marker for visualization in RViz: -->
+    <visual>
+      <geometry>
+        <sphere radius="0.005"/>  <!-- 5mm sphere marker -->
+      </geometry>
+      <material name="tcp_marker">
+        <color rgba="1 0 0 1"/>  <!-- Red color -->
+      </material>
+    </visual>
+  </link>
+  <!-- Fixed joint connecting base to TCP at desired offset -->
+  <joint name="${name}_tcp_joint" type="fixed">
+    <parent link="${name}_base"/>
+    <child link="${name}_tcp"/>
+    <!-- Position TCP 65mm forward and centered between fingers -->
+    <origin xyz="0.0 0.05 0.13" rpy="0 0 0"/>
+  </joint>
      <!--Extensions -->
     <xacro:yumi_servo_gripper_gazebo name="${name}" />

File: yumi_description/urdf/yumi.urdf (robot description, URDF)
Before this commit: robot yumi, 23 links, 22 joints
Links:
- added link gripper_l_tcp; visual sphere radius=0.005
- added link gripper_r_tcp; visual sphere radius=0.005
Joints:
- added joint gripper_l_tcp_joint: type fixed, parent gripper_l_base, child gripper_l_tcp, origin xyz=0.0 0.05 0.13 rpy=0 0 0
- added joint gripper_r_tcp_joint: type fixed, parent gripper_r_base, child gripper_r_tcp, origin xyz=0.0 0.05 0.13 rpy=0 0 0
