Commit message: Add SPL eurocontainer/redboard slots, grippers with custom fingers, and left/right layout
- spl_electricalstation_slots.xacro: add left/right (+y/-y) side tagging
  to eurocontainer_slot and redboard_slot macros; slot marker boxes are
  now 1cm thin boxes sitting flush with the table top (link raised 1cm
  above table_top, box drawn below the link origin).
- spl_redboard.xacro: real Redboard mesh marker macro (spl_markers
  UNP_SPL_Redboard.obj), mounted on redboard slots.
- spl_eurocontainer.xacro (new): real Eurocontainer mesh marker macro
  (spl_markers EuroContainer_EG43-12HG.stl, rotated 90deg about X),
  simplified 40x30x12cm box collision, and a 40-slot SPL layout (4
  sub-grids of 2x5, arranged 2x2 across the footprint, 2cm edge inset,
  10.15cm column / 2cm row pitch within each sub-grid).
- spl_yumi_servo_gripper.xacro (new): SPL-scoped copy of
  yumi_description's yumi_servo_gripper macro, using the custom SPL
  finger meshes (UNP_SPL_YumiLeftFinger_v2.3.stl /
  UNP_SPL_YumiRightFinger_v2.3.stl) instead of the stock finger mesh;
  right finger visual/collision rotated 180deg about Z. Keeps
  yumi_description package untouched/generic.
- spl_electricalstation.xacro: instantiate both left/right eurocontainer
  and redboard slots, the new SPL grippers on yumi_link_7_r/l, and the
  new SPL eurocontainer mesh markers.
- Add MODUL4R table mesh and SPL finger meshes to
  spl_electricalstation_description/meshes, and the EuroContainer mesh
  to spl_markers/meshes.

File: spl_electricalstation_description/urdf/spl_electricalstation.xacro (robot description, xacro)
@@ -6,22 +6,40 @@
   <!-- Define PI in case utilities.xacro is not available in some include orders -->
   <xacro:property name="PI" value="3.141592653589793"/>
-  <!-- Table dimensions -->
-  <xacro:property name="table_length" value="1.2"/>
+  <!-- Table dimensions.
+       Matches the real MODUL4R_YumiWheeledSupport_noWheels.dae mesh, as
+       used (and offset) in MODUL4R/ROS/ros_modules/modular-description/
+       modul4r_station_description/urdf/modul4r_station.urdf.xacro:
+       that reference file's own collision box for this same mesh is
+       "<box size="0.8 0.8 0.01"/>" at origin xyz="-0.4 0 0.9", i.e. the
+       mesh's footprint is NOT centered on the link origin: it spans
+       roughly x in [-0.8, 0], y in [-0.4, 0.4], height ~0.9 m, with the
+       link/mesh origin at one corner (x=0 edge), not the footprint center. -->
+  <xacro:property name="table_length" value="0.8"/>
   <xacro:property name="table_width" value="0.8"/>
-  <xacro:property name="table_height" value="0.7"/>
-  <!-- Table / base_link as a simple box. The link origin (0,0,0) is the CENTER of the box,
-       so the top surface of the table sits at z = table_height/2. -->
+  <xacro:property name="table_height" value="0.9"/>
+  <!-- x-offset of the collision box center relative to the mesh/link
+       origin, matching the reference modul4r_station.urdf.xacro. -->
+  <xacro:property name="table_collision_offset_x" value="-0.4"/>
+  <!-- Instead of offsetting yumi off table_top, we keep yumi at table_top's
+       origin (0,0,0) and shift the table mesh (visual + collision) the
+       other way by half of the reference's yumi offset (0.21 / 2 = 0.105),
+       so that yumi ends up positioned the same relative to the table mesh
+       as in the reference file, without yumi itself being offset. -->
+  <xacro:property name="table_mesh_offset_x" value="0.105"/>
+  <!-- Table / base_link: visual is the real support mesh, shifted by
+       table_mesh_offset_x (see above). Collision is a simple box of the
+       same footprint/height for fast collision checking, offset in x to
+       match the mesh's actual footprint (table_collision_offset_x) plus
+       the same table_mesh_offset_x shift, and centered in z from the
+       mesh's bottom (z=0) up to table_height. -->
   <link name="base_link">
     <visual>
-      <origin xyz="0 0 ${table_height / 2}" rpy="0 0 0"/>
+      <origin xyz="${table_mesh_offset_x} 0 0" rpy="0 0 0"/>
       <geometry>
-        <box size="${table_length} ${table_width} ${table_height}" />
+        <mesh filename="package://spl_electricalstation_description/meshes/MODUL4R_YumiWheeledSupport_noWheels.dae" scale="1 1 1"/>
       </geometry>
-      <material name="Brown">
-        <color rgba="0.6 0.4 0.2 1.0"/>
-      </material>
     </visual>
     <collision>
-      <origin xyz="0 0 ${table_height / 2}" rpy="0 0 0"/>
+      <origin xyz="${table_collision_offset_x + table_mesh_offset_x} 0 ${table_height / 2}" rpy="0 0 0"/>
       <geometry>
         <box size="${table_length} ${table_width} ${table_height}" />
@@ -29,5 +47,5 @@
     </collision>
     <inertial>
-      <origin xyz="0 0 ${table_height / 2}" rpy="0 0 0"/>
+      <origin xyz="${table_collision_offset_x + table_mesh_offset_x} 0 ${table_height / 2}" rpy="0 0 0"/>
       <mass value="20.0"/>
       <inertia ixx="1" ixy="0" ixz="0" iyy="1" iyz="0" izz="1"/>
@@ -65,10 +83,33 @@
   <!-- Include the yumi_description xacro and attach it to table_top -->
   <xacro:include filename="$(find yumi_description)/urdf/yumi.xacro" />
-  <!-- Call the yumi macro. The yumi macro signature is: parent name hardware_interface *origin -->
-  <!-- yumi_base_link is spawned at table_top's frame (already at the table surface), so no extra offset needed. -->
+  <!-- NOTE: the "parent"/"*origin" params of the xacro:yumi macro are NOT
+       actually used by the macro itself (yumi_base_link is defined
+       standalone inside it); the real attachment is the explicit fixed
+       joint below. Unlike the reference modul4r_station.urdf.xacro
+       (which offsets yumi_base_link by xyz="-0.21 0.0 0.905" relative to
+       its mesh/base link origin), we keep yumi_base_link centered at
+       table_top's origin (0,0,0) and instead shift the table mesh the
+       other way (see table_mesh_offset_x above), so yumi stays at a
+       clean 0,0 while ending up correctly positioned relative to the
+       table mesh. -->
   <xacro:yumi parent="table_top" name="yumi" hardware_interface="">
     <origin xyz="0 0 0" rpy="0 0 0" />
   </xacro:yumi>
-  <!-- Attach the yumi base directly on the table surface (table_top), single root remains base_link -->
+  <!-- Include and instantiate the SPL servo grippers (with SPL-specific
+       finger meshes) on each arm's wrist link (yumi_link_7_r / yumi_link_7_l),
+       matching the origin used by yumi_description's yumi.urdf.xacro
+       reference (0 0 0.007, rotated 180 deg about z). This uses a local
+       spl_yumi_servo_gripper macro (spl_yumi_servo_gripper.xacro) instead
+       of yumi_description's generic gripper, so yumi_description itself
+       stays untouched. -->
+  <xacro:include filename="$(find spl_electricalstation_description)/urdf/spl_yumi_servo_gripper.xacro" />
+  <xacro:spl_yumi_servo_gripper name="gripper_r" hardware_interface="" parent="yumi_link_7_r">
+    <origin xyz="0 0 0.007" rpy="0 0 ${PI}" />
+  </xacro:spl_yumi_servo_gripper>
+  <xacro:spl_yumi_servo_gripper name="gripper_l" hardware_interface="" parent="yumi_link_7_l">
+    <origin xyz="0 0 0.007" rpy="0 0 ${PI}" />
+  </xacro:spl_yumi_servo_gripper>
+  <!-- Attach the yumi base on the table surface (table_top) at its origin.
+       Single root remains base_link. -->
   <joint name="table_top_to_yumi_base_link" type="fixed">
     <parent link="table_top"/>
@@ -79,3 +120,21 @@
   <xacro:include filename="$(find spl_electricalstation_description)/urdf/spl_electricalstation_slots.xacro" />
   <xacro:electrical_station_slots parent="table_top" />
+  <!-- Include and instantiate the real Eurocontainer mesh markers (with
+       their 2x5 grid of SPL slot frames) on the left and right
+       eurocontainer slots. -->
+  <xacro:include filename="$(find spl_electricalstation_description)/urdf/spl_eurocontainer.xacro" />
+  <xacro:spl_eurocontainer parent="eurocontainer_slot_left" name="left"/>
+  <xacro:spl_eurocontainer parent="eurocontainer_slot_right" name="right"/>
+  <!-- Include and instantiate the real Redboard mesh markers on each
+       left-side (+y) slot, named 00-07 to match the Isaac Sim object naming
+       (raster order: row0 col0..3 -> 00-03, row1 col0..3 -> 04-07). -->
+  <xacro:include filename="$(find spl_electricalstation_description)/urdf/spl_redboard.xacro" />
+  <xacro:spl_redboard parent="redboard_slot_left_0_0" name="'00'"/>
+  <xacro:spl_redboard parent="redboard_slot_left_0_1" name="'01'"/>
+  <xacro:spl_redboard parent="redboard_slot_left_0_2" name="'02'"/>
+  <xacro:spl_redboard parent="redboard_slot_left_0_3" name="'03'"/>
+  <xacro:spl_redboard parent="redboard_slot_left_1_0" name="'04'"/>
+  <xacro:spl_redboard parent="redboard_slot_left_1_1" name="'05'"/>
+  <xacro:spl_redboard parent="redboard_slot_left_1_2" name="'06'"/>
+  <xacro:spl_redboard parent="redboard_slot_left_1_3" name="'07'"/>
 </robot>

File: spl_electricalstation_description/urdf/spl_electricalstation_slots.xacro (robot description, xacro)
@@ -14,28 +14,46 @@
   <xacro:property name="eurocontainer_width"  value="0.30"/> <!-- y -->
   <xacro:property name="eurocontainer_height" value="0.12"/> <!-- z -->
-  <!-- Position of the Eurocontainer slot center, relative to table_top -->
-  <xacro:property name="eurocontainer_offset_x" value="0.45"/>
-  <xacro:property name="eurocontainer_offset_y" value="0.0"/>
+  <!-- Position of the Eurocontainer slot center, relative to table_top.
+       eurocontainer_offset_y is the middle point between the two
+       recovered Isaac Sim ground-truth y values (eurocontainer00 y=0.15,
+       eurocontainer01 y=0.35 -> midpoint 0.25), used as the |y| magnitude
+       for both the left (+y) and right (-y) instances below. -->
+  <xacro:property name="eurocontainer_offset_x" value="0.55"/>
+  <xacro:property name="eurocontainer_offset_y" value="0.20"/>
   <!-- Redboard slots -->
-  <!-- 8 slots arranged in 2 rows x 4 columns, to the left of the robot (+y) -->
+  <!-- 8 slots arranged in 2 rows x 4 columns, to the side of the robot -->
   <xacro:property name="redboard_length" value="0.10"/> <!-- x (placeholder board size) -->
   <xacro:property name="redboard_width"  value="0.08"/> <!-- y (placeholder board size) -->
   <xacro:property name="redboard_height" value="0.02"/> <!-- z (placeholder board thickness) -->
-  <xacro:property name="redboard_spacing_x" value="0.15"/> <!-- column pitch along x -->
-  <xacro:property name="redboard_spacing_y" value="0.14"/> <!-- row pitch along y -->
+  <!-- Spacing and origin match recovered Isaac Sim ground-truth poses
+       (isaac_sim_objects.json, leftarm/position/redboard_XX, frame_id "world",
+       assumed coincident with the robot base / table_top, no additional offset).
+       redboard_origin_y / redboard_spacing_y are used as |y| magnitudes for
+       both the left (+y) and right (-y) instances below. -->
+  <xacro:property name="redboard_spacing_x" value="0.14"/> <!-- column pitch along x -->
+  <xacro:property name="redboard_spacing_y" value="0.15"/> <!-- row pitch along y -->
   <!-- Position of the first (row0,col0) redboard slot, relative to table_top -->
-  <xacro:property name="redboard_origin_x" value="-0.20"/>
-  <xacro:property name="redboard_origin_y" value="0.25"/>
+  <xacro:property name="redboard_origin_x" value="-0.15"/>
+  <xacro:property name="redboard_origin_y" value="0.40"/>
+  <!-- All slot marker boxes (eurocontainer and redboard) are thin 1 cm
+       high boxes, drawn BELOW their link's origin (i.e. from z=-slot_marker_height
+       to z=0). The slot link itself is raised slot_link_height_above_table
+       (1 cm) above table_top via the parent joint, so the box's top face
+       sits flush with the table surface. -->
+  <xacro:property name="slot_marker_height" value="0.01"/>
+  <xacro:property name="slot_link_height_above_table" value="0.01"/>
   <!-- ===================================================================
        Macro: eurocontainer_slot
        Creates a thin, semi-transparent box link marking where the
        Eurocontainer should be placed, and a fixed joint to "parent".
+       "side" is either "left" or "right" and only affects the link name
+       (the y value passed in should already carry the correct sign).
   =================================================================== -->
-  <xacro:macro name="eurocontainer_slot" params="parent name x y">
+  <xacro:macro name="eurocontainer_slot" params="parent name side x y">
     <link name="${name}">
       <visual>
-        <origin xyz="0 0 ${eurocontainer_height / 2}" rpy="0 0 0"/>
+        <origin xyz="0 0 ${-slot_marker_height / 2}" rpy="0 0 0"/>
         <geometry>
-          <box size="${eurocontainer_length} ${eurocontainer_width} ${eurocontainer_height}"/>
+          <box size="${eurocontainer_length} ${eurocontainer_width} ${slot_marker_height}"/>
         </geometry>
         <material name="EuroContainerBlue">
@@ -44,11 +62,11 @@
       </visual>
       <collision>
-        <origin xyz="0 0 ${eurocontainer_height / 2}" rpy="0 0 0"/>
+        <origin xyz="0 0 ${-slot_marker_height / 2}" rpy="0 0 0"/>
         <geometry>
-          <box size="${eurocontainer_length} ${eurocontainer_width} ${eurocontainer_height}"/>
+          <box size="${eurocontainer_length} ${eurocontainer_width} ${slot_marker_height}"/>
         </geometry>
       </collision>
       <inertial>
-        <origin xyz="0 0 ${eurocontainer_height / 2}" rpy="0 0 0"/>
+        <origin xyz="0 0 ${-slot_marker_height / 2}" rpy="0 0 0"/>
         <mass value="0.01"/>
         <inertia ixx="0.0001" ixy="0" ixz="0" iyy="0.0001" iyz="0" izz="0.0001"/>
@@ -58,5 +76,5 @@
       <parent link="${parent}"/>
       <child link="${name}"/>
-      <origin xyz="${x} ${y} 0" rpy="0 0 0"/>
+      <origin xyz="${x} ${y} ${slot_link_height_above_table}" rpy="0 0 0"/>
     </joint>
   </xacro:macro>
@@ -65,11 +83,13 @@
        Creates a thin box link marking a single Redboard slot, and a
        fixed joint to "parent".
+       "side" is either "left" or "right" and only affects the link name
+       (the y value passed in should already carry the correct sign).
   =================================================================== -->
-  <xacro:macro name="redboard_slot" params="parent name x y">
+  <xacro:macro name="redboard_slot" params="parent name side x y">
     <link name="${name}">
       <visual>
-        <origin xyz="0 0 ${redboard_height / 2}" rpy="0 0 0"/>
+        <origin xyz="0 0 ${-slot_marker_height / 2}" rpy="0 0 0"/>
         <geometry>
-          <box size="${redboard_length} ${redboard_width} ${redboard_height}"/>
+          <box size="${redboard_length} ${redboard_width} ${slot_marker_height}"/>
         </geometry>
         <material name="RedboardGreen">
@@ -78,11 +98,11 @@
       </visual>
       <collision>
-        <origin xyz="0 0 ${redboard_height / 2}" rpy="0 0 0"/>
+        <origin xyz="0 0 ${-slot_marker_height / 2}" rpy="0 0 0"/>
         <geometry>
-          <box size="${redboard_length} ${redboard_width} ${redboard_height}"/>
+          <box size="${redboard_length} ${redboard_width} ${slot_marker_height}"/>
         </geometry>
       </collision>
       <inertial>
-        <origin xyz="0 0 ${redboard_height / 2}" rpy="0 0 0"/>
+        <origin xyz="0 0 ${-slot_marker_height / 2}" rpy="0 0 0"/>
         <mass value="0.01"/>
         <inertia ixx="0.0001" ixy="0" ixz="0" iyy="0.0001" iyz="0" izz="0.0001"/>
@@ -92,5 +112,5 @@
       <parent link="${parent}"/>
       <child link="${name}"/>
-      <origin xyz="${x} ${y} 0" rpy="0 0 0"/>
+      <origin xyz="${x} ${y} ${slot_link_height_above_table}" rpy="0 0 0"/>
     </joint>
   </xacro:macro>
@@ -98,35 +118,64 @@
        Macro: electrical_station_slots
        Instantiates the Eurocontainer slot and all 8 Redboard slots
-       (2 rows x 4 columns) on the given parent link (typically "table_top").
+       (2 rows x 4 columns), mirrored for both the left (+y) arm side and
+       the right (-y) arm side, on the given parent link (typically
+       "table_top").
   =================================================================== -->
   <xacro:macro name="electrical_station_slots" params="parent">
-    <xacro:eurocontainer_slot parent="${parent}" name="eurocontainer_slot"
+    <!-- Eurocontainer: left (+y) and right (-y) -->
+    <xacro:eurocontainer_slot parent="${parent}" name="eurocontainer_slot_left" side="left"
                                x="${eurocontainer_offset_x}" y="${eurocontainer_offset_y}"/>
-    <!-- Row 0 (y = redboard_origin_y) -->
-    <xacro:redboard_slot parent="${parent}" name="redboard_slot_0_0"
+    <xacro:eurocontainer_slot parent="${parent}" name="eurocontainer_slot_right" side="right"
+                               x="${eurocontainer_offset_x}" y="${-eurocontainer_offset_y}"/>
+    <!-- Redboards: left (+y) -->
+    <xacro:redboard_slot parent="${parent}" name="redboard_slot_left_0_0" side="left"
                           x="${redboard_origin_x + 0 * redboard_spacing_x}"
                           y="${redboard_origin_y + 0 * redboard_spacing_y}"/>
-    <xacro:redboard_slot parent="${parent}" name="redboard_slot_0_1"
+    <xacro:redboard_slot parent="${parent}" name="redboard_slot_left_0_1" side="left"
                           x="${redboard_origin_x + 1 * redboard_spacing_x}"
                           y="${redboard_origin_y + 0 * redboard_spacing_y}"/>
-    <xacro:redboard_slot parent="${parent}" name="redboard_slot_0_2"
+    <xacro:redboard_slot parent="${parent}" name="redboard_slot_left_0_2" side="left"
                           x="${redboard_origin_x + 2 * redboard_spacing_x}"
                           y="${redboard_origin_y + 0 * redboard_spacing_y}"/>
-    <xacro:redboard_slot parent="${parent}" name="redboard_slot_0_3"
+    <xacro:redboard_slot parent="${parent}" name="redboard_slot_left_0_3" side="left"
                           x="${redboard_origin_x + 3 * redboard_spacing_x}"
                           y="${redboard_origin_y + 0 * redboard_spacing_y}"/>
-    <!-- Row 1 (y = redboard_origin_y + redboard_spacing_y) -->
-    <xacro:redboard_slot parent="${parent}" name="redboard_slot_1_0"
+    <xacro:redboard_slot parent="${parent}" name="redboard_slot_left_1_0" side="left"
                           x="${redboard_origin_x + 0 * redboard_spacing_x}"
                           y="${redboard_origin_y + 1 * redboard_spacing_y}"/>
-    <xacro:redboard_slot parent="${parent}" name="redboard_slot_1_1"
+    <xacro:redboard_slot parent="${parent}" name="redboard_slot_left_1_1" side="left"
                           x="${redboard_origin_x + 1 * redboard_spacing_x}"
                           y="${redboard_origin_y + 1 * redboard_spacing_y}"/>
-    <xacro:redboard_slot parent="${parent}" name="redboard_slot_1_2"
+    <xacro:redboard_slot parent="${parent}" name="redboard_slot_left_1_2" side="left"
                           x="${redboard_origin_x + 2 * redboard_spacing_x}"
                           y="${redboard_origin_y + 1 * redboard_spacing_y}"/>
-    <xacro:redboard_slot parent="${parent}" name="redboard_slot_1_3"
+    <xacro:redboard_slot parent="${parent}" name="redboard_slot_left_1_3" side="left"
                           x="${redboard_origin_x + 3 * redboard_spacing_x}"
                           y="${redboard_origin_y + 1 * redboard_spacing_y}"/>
+    <!-- Redboards: right (-y), mirror of the left layout -->
+    <xacro:redboard_slot parent="${parent}" name="redboard_slot_right_0_0" side="right"
+                          x="${redboard_origin_x + 0 * redboard_spacing_x}"
+                          y="${-(redboard_origin_y + 0 * redboard_spacing_y)}"/>
+    <xacro:redboard_slot parent="${parent}" name="redboard_slot_right_0_1" side="right"
+                          x="${redboard_origin_x + 1 * redboard_spacing_x}"
+                          y="${-(redboard_origin_y + 0 * redboard_spacing_y)}"/>
+    <xacro:redboard_slot parent="${parent}" name="redboard_slot_right_0_2" side="right"
+                          x="${redboard_origin_x + 2 * redboard_spacing_x}"
+                          y="${-(redboard_origin_y + 0 * redboard_spacing_y)}"/>
+    <xacro:redboard_slot parent="${parent}" name="redboard_slot_right_0_3" side="right"
+                          x="${redboard_origin_x + 3 * redboard_spacing_x}"
+                          y="${-(redboard_origin_y + 0 * redboard_spacing_y)}"/>
+    <xacro:redboard_slot parent="${parent}" name="redboard_slot_right_1_0" side="right"
+                          x="${redboard_origin_x + 0 * redboard_spacing_x}"
+                          y="${-(redboard_origin_y + 1 * redboard_spacing_y)}"/>
+    <xacro:redboard_slot parent="${parent}" name="redboard_slot_right_1_1" side="right"
+                          x="${redboard_origin_x + 1 * redboard_spacing_x}"
+                          y="${-(redboard_origin_y + 1 * redboard_spacing_y)}"/>
+    <xacro:redboard_slot parent="${parent}" name="redboard_slot_right_1_2" side="right"
+                          x="${redboard_origin_x + 2 * redboard_spacing_x}"
+                          y="${-(redboard_origin_y + 1 * redboard_spacing_y)}"/>
+    <xacro:redboard_slot parent="${parent}" name="redboard_slot_right_1_3" side="right"
+                          x="${redboard_origin_x + 3 * redboard_spacing_x}"
+                          y="${-(redboard_origin_y + 1 * redboard_spacing_y)}"/>
   </xacro:macro>
 </robot>

File: yumi_description/urdf/yumi.urdf (robot description, URDF)
Before this commit: robot yumi, 25 links, 24 joints
Links:
- link gripper_l_finger_l: geometry collision mesh filename=package://spl_electricalstation_description/meshes/UNP_SPL_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; visual mesh filename=package://spl_electricalstation_description/meshes/UNP_SPL_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
- link gripper_l_finger_r: geometry collision mesh filename=package://spl_electricalstation_description/meshes/UNP_SPL_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; visual mesh filename=package://spl_electricalstation_description/meshes/UNP_SPL_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
- link gripper_r_finger_l: geometry collision mesh filename=package://spl_electricalstation_description/meshes/UNP_SPL_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; visual mesh filename=package://spl_electricalstation_description/meshes/UNP_SPL_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
- link gripper_r_finger_r: geometry collision mesh filename=package://spl_electricalstation_description/meshes/UNP_SPL_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; visual mesh filename=package://spl_electricalstation_description/meshes/UNP_SPL_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
