Commit message: Add SPL eurocontainer/redboard slots, grippers with custom fingers, and left/right layout
- spl_electricalstation_slots.xacro: add left/right (+y/-y) side tagging
  to eurocontainer_slot and redboard_slot macros; slot marker boxes are
  now 1cm thin boxes sitting flush with the table top (link raised 1cm
  above table_top, box drawn below the link origin).
- spl_redboard.xacro: real Redboard mesh marker macro (spl_markers
  UNP_SPL_Redboard.obj), mounted on redboard slots.
- spl_eurocontainer.xacro (new): real Eurocontainer mesh marker macro
  (spl_markers EuroContainer_EG43-12HG.stl, rotated 90deg about X),
  simplified 40x30x12cm box collision, and a 40-slot SPL layout (4
  sub-grids of 2x5, arranged 2x2 across the footprint, 2cm edge inset,
  10.15cm column / 2cm row pitch within each sub-grid).
- spl_yumi_servo_gripper.xacro (new): SPL-scoped copy of
  yumi_description's yumi_servo_gripper macro, using the custom SPL
  finger meshes (UNP_SPL_YumiLeftFinger_v2.3.stl /
  UNP_SPL_YumiRightFinger_v2.3.stl) instead of the stock finger mesh;
  right finger visual/collision rotated 180deg about Z. Keeps
  yumi_description package untouched/generic.
- spl_electricalstation.xacro: instantiate both left/right eurocontainer
  and redboard slots, the new SPL grippers on yumi_link_7_r/l, and the
  new SPL eurocontainer mesh markers.
- Add MODUL4R table mesh and SPL finger meshes to
  spl_electricalstation_description/meshes, and the EuroContainer mesh
  to spl_markers/meshes.

File: yumi_moveit_config/config/gazebo_yumi.urdf (robot description, URDF)
Before this commit: robot yumi, 23 links, 22 joints
Links:
- link gripper_l_finger_l: geometry collision mesh filename=package://spl_electricalstation_description/meshes/UNP_SPL_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; visual mesh filename=package://spl_electricalstation_description/meshes/UNP_SPL_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
- link gripper_l_finger_r: geometry collision mesh filename=package://spl_electricalstation_description/meshes/UNP_SPL_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; visual mesh filename=package://spl_electricalstation_description/meshes/UNP_SPL_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
- link gripper_r_finger_l: geometry collision mesh filename=package://spl_electricalstation_description/meshes/UNP_SPL_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; visual mesh filename=package://spl_electricalstation_description/meshes/UNP_SPL_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
- link gripper_r_finger_r: geometry collision mesh filename=package://spl_electricalstation_description/meshes/UNP_SPL_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; visual mesh filename=package://spl_electricalstation_description/meshes/UNP_SPL_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
